Commit message: added a equivalent rotor with joint to the motor.urdf

File: motor_description/urdf/motor.urdf (robot description, URDF)
Before this commit: robot motor, 3 links, 2 joints
Links:
- link base_link: mass None -> 0.1; geometry collision box size=0.1 0.1 0.01; visual box size=0.1 0.1 0.01
- link rotor: mass None -> 0.1; geometry collision cylinder length=0.055 radius=0.009; visual cylinder length=0.055 radius=0.009
Joints:
- joint motor_axis: axis 1 0 0 -> 0 0 1; origin xyz=0 0 0.1 -> xyz=0 0 0.1 rpy=0 1.570796327 0

Commit message: added details to the motor-model, work in progress state

File: motor_description/urdf/motor.urdf (robot description, URDF)
Before this commit: robot motor, 3 links, 2 joints
Links:
- added link flywheel, mass 0.37; collision cylinder length=0.006 radius=0.048; visual cylinder length=0.006 radius=0.048
- link base_link: mass 0.1 -> 1
- link rotor: mass 0.1 -> 0.13
Joints:
- added joint coupling: type fixed, parent rotor, child flywheel, origin xyz=0 0 0.1
