Commit message: change urdf

File: motor_description/urdf/motor_eeros.urdf (robot description, URDF)
Before this commit: robot motor, 4 links, 3 joints
Links:
- removed link rotor
- added link damper, mass 0.13; collision cylinder length=0.055 radius=0.009; visual cylinder length=0.055 radius=0.009
- added link motor, mass 0.13; collision cylinder length=0.055 radius=0.009; visual cylinder length=0.055 radius=0.009
- link base_link: geometry collision box size=0.1 0.1 0.01; visual box size=0.2 0.1 0.01
Joints:
- added joint damper_axis: type continuous, parent base_link, child damper, origin xyz=-0.07 0 0.1 rpy=0 0 0, axis 1 0 0
- joint coupling: axis (none) -> 1 0 0; origin xyz=0 0 0.1 -> xyz=-0.09 0 0 rpy=0 0 0; parent rotor -> motor; type fixed -> continuous
- joint motor_axis: axis 0 0 1 -> 1 0 0; child rotor -> motor; origin xyz=0 0 0.1 rpy=0 1.570796327 0 -> xyz=0.07 0 0.1 rpy=0 0 0

Commit message: close kinematic chain

File: motor_description/urdf/motor_eeros.urdf (robot description, URDF)
Before this commit: robot motor, 5 links, 4 joints
Joints:
- joint coupling: axis 1 0 0 -> (none); type continuous -> fixed
- joint damper_axis: mimic (none) -> joint=motor_axis multiplier=1 offset=0

Commit message: changed urdf

File: motor_description/urdf/motor_eeros.urdf (robot description, URDF)
Before this commit: robot motor, 5 links, 4 joints
Joints:
- joint fixe_base: origin xyz=0 0 0.005 -> xyz=0 0 0.005 rpy=0 0 0
